Commit message: feat: 添加 Agibot D1 和 XSDog 任务的观测项维度说明及训练配置

File: source/robot_lab/data/Robots/etc/xsdog_description/urdf.urdf (robot description, URDF)
Before this commit: robot urdf, 17 links, 16 joints
Joints:
- joint lf_calf: limit lower=-2.787 upper=-0.9203 effort=0 velocity=0 -> lower=-2.787 upper=-0.9203 effort=110 velocity=30
- joint lf_hip: limit lower=-0.785 upper=0.785 effort=0 velocity=0 -> lower=-0.785 upper=0.785 effort=110 velocity=30
- joint lf_thigh: limit lower=-1.222 upper=2.793 effort=0 velocity=0 -> lower=-1.222 upper=2.793 effort=110 velocity=30
- joint lh_calf: limit lower=-2.787 upper=-0.9203 effort=0 velocity=0 -> lower=-2.787 upper=-0.9203 effort=110 velocity=30
- joint lh_hip: limit lower=-0.785 upper=0.785 effort=0 velocity=0 -> lower=-0.785 upper=0.785 effort=110 velocity=30
- joint lh_thigh: limit lower=-1.222 upper=2.793 effort=0 velocity=0 -> lower=-1.222 upper=2.793 effort=110 velocity=30
- joint rf_calf: limit lower=-2.787 upper=-0.9203 effort=0 velocity=0 -> lower=-2.787 upper=-0.9203 effort=110 velocity=30
- joint rf_hip: limit lower=-0.785 upper=0.785 effort=0 velocity=0 -> lower=-0.785 upper=0.785 effort=110 velocity=30
- joint rf_thigh: limit lower=-1.222 upper=2.793 effort=0 velocity=0 -> lower=-1.222 upper=2.793 effort=110 velocity=30
- joint rh_calf: limit lower=-2.787 upper=-0.9203 effort=0 velocity=0 -> lower=-2.787 upper=-0.9203 effort=110 velocity=30
- joint rh_hip: limit lower=-0.785 upper=0.785 effort=0 velocity=0 -> lower=-0.785 upper=0.785 effort=110 velocity=30
- joint rh_thigh: limit lower=-1.222 upper=2.793 effort=0 velocity=0 -> lower=-1.222 upper=2.793 effort=110 velocity=30
